File: PandaSat_Payload.sch (EAGLE design)
At the start: 16 parts, among them J1 U.FL, J4 FEMALE 2x3, J5 U.FL, J6 FEMALE 2x3, U1 CH340G, U12 EP2W+, U14 S1216V8, Y1 12MHz

Commit message: Added new Eagle Files for payload board
-modified pins USB socket
-added 4 pins connector (socket - Pi)
Parts:
- added J7: (no value), SparkFun-Connectors:CONN_04
Connections:
- new net N$3: PCB1.GND@20
- net D+: now also J7.3, X1.3; no longer X1.2
- net D-: now also J7.2, X1.2; no longer X1.3
- net GND: now also J7.4, PCB1.GND@14, PCB1.GND@25, PCB1.GND@30, PCB1.GND@34, PCB1.GND@39, PCB1.GND@6, X1.4; no longer X1.1
- net VCC5: now also J7.1, X1.1; no longer X1.4
Other:
- note added: "SDR (Socket Connector)"
Changed lines of the file:
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@@
 <part name="J3" library="SparkFun-Connectors" deviceset="CONN_04" device=""/>
 <part name="J4" library="SparkFun-Connectors" deviceset="CONN_03X2" device="FEMALE" value="FEMALE 2x3"/>
+<part name="J7" library="SparkFun-Connectors" deviceset="CONN_04" device=""/>
 </parts>
 <sheets>
@@
 </segment>
 <segment>
-<pinref part="X1" gate="G$1" pin="1"/>
-<wire x1="121.92" y1="30.48" x2="134.62" y2="30.48" width="0.1524" layer="91"/>
-<label x="134.62" y="30.48" size="1.4224" layer="95" xref="yes"/>
-</segment>
-<segment>
 <pinref part="J6" gate="G$1" pin="3"/>
 <wire x1="185.42" y1="58.42" x2="172.72" y2="58.42" width="0.1524" layer="91"/>
@@
 <wire x1="215.9" y1="104.14" x2="220.98" y2="104.14" width="0.1524" layer="91"/>
 <label x="220.98" y="104.14" size="1.778" layer="95" xref="yes"/>
+</segment>
+<segment>
+<pinref part="PCB1" gate="G$1" pin="GND@6"/>
+<wire x1="106.68" y1="152.4" x2="132.08" y2="152.4" width="0.1524" layer="91"/>
+<label x="132.08" y="152.4" size="1.778" layer="95" xref="yes"/>
+</segment>
+<segment>
+<pinref part="PCB1" gate="G$1" pin="GND@14"/>
+<wire x1="106.68" y1="132.08" x2="132.08" y2="132.08" width="0.1524" layer="91"/>
+<label x="132.08" y="132.08" size="1.778" layer="95" xref="yes"/>
+</segment>
+<segment>
+<pinref part="PCB1" gate="G$1" pin="GND@25"/>
+<wire x1="78.74" y1="101.6" x2="78.74" y2="99.06" width="0.1524" layer="91"/>
+<wire x1="78.74" y1="99.06" x2="132.08" y2="99.06" width="0.1524" layer="91"/>
+<label x="132.08" y="99.06" size="1.778" layer="95" xref="yes"/>
+</segment>
+<segment>
+<pinref part="PCB1" gate="G$1" pin="GND@30"/>
+<wire x1="106.68" y1="91.44" x2="132.08" y2="91.44" width="0.1524" layer="91"/>
+<label x="132.08" y="91.44" size="1.778" layer="95" xref="yes"/>
+</segment>
+<segment>
+<pinref part="PCB1" gate="G$1" pin="GND@34"/>
+<wire x1="106.68" y1="81.28" x2="132.08" y2="81.28" width="0.1524" layer="91"/>
+<label x="132.08" y="81.28" size="1.778" layer="95" xref="yes"/>
+</segment>
+<segment>
+<pinref part="PCB1" gate="G$1" pin="GND@39"/>
+<wire x1="78.74" y1="66.04" x2="78.74" y2="60.96" width="0.1524" layer="91"/>
+<wire x1="78.74" y1="60.96" x2="132.08" y2="60.96" width="0.1524" layer="91"/>
+<label x="132.08" y="60.96" size="1.778" layer="95" xref="yes"/>
+</segment>
+<segment>
+<pinref part="X1" gate="G$1" pin="4"/>
+<wire x1="121.92" y1="38.1" x2="134.62" y2="38.1" width="0.1524" layer="91"/>
+<label x="134.62" y="38.1" size="1.4224" layer="95" xref="yes"/>
 </segment>
 </net>
@@
 </segment>
 <segment>
-<pinref part="X1" gate="G$1" pin="4"/>
-<wire x1="121.92" y1="38.1" x2="134.62" y2="38.1" width="0.1524" layer="91"/>
-<label x="134.62" y="38.1" size="1.4224" layer="95" xref="yes"/>
-</segment>
-<segment>
 <pinref part="J6" gate="G$1" pin="1"/>
 <wire x1="185.42" y1="60.96" x2="167.64" y2="60.96" width="0.1524" layer="91"/>
 <label x="167.64" y="60.96" size="1.016" layer="95" xref="yes"/>
 </segment>
+<segment>
+<pinref part="X1" gate="G$1" pin="1"/>
+<wire x1="121.92" y1="30.48" x2="134.62" y2="30.48" width="0.1524" layer="91"/>
+<label x="134.62" y="30.48" size="1.4224" layer="95" xref="yes"/>
+</segment>
 </net>
 <net name="UART2_RX" class="0">
@@
 </segment>
 </net>
-<net name="D-" class="0">
+<net name="D+" class="0">
 <segment>
 <pinref part="X1" gate="G$1" pin="3"/>
@@
 </segment>
 </net>
-<net name="D+" class="0">
+<net name="GPS_CLK" class="0">
+<segment>
+<pinref part="U14" gate="G$1" pin="1PPS"/>
+<wire x1="210.82" y1="144.78" x2="226.06" y2="144.78" width="0.1524" layer="91"/>
+<label x="226.06" y="144.78" size="1.4224" layer="95" xref="yes"/>
+</segment>
+<segment>
+<pinref part="PCB1" gate="G$1" pin="GPIO24"/>
+<wire x1="106.68" y1="121.92" x2="132.08" y2="121.92" width="0.1524" layer="91"/>
+<label x="132.08" y="121.92" size="1.4224" layer="95" xref="yes"/>
+</segment>
+</net>
+<net name="ENABLE1" class="0">
+<segment>
+<pinref part="PCB1" gate="G$1" pin="GPIO18"/>
+<wire x1="106.68" y1="137.16" x2="132.08" y2="137.16" width="0.1524" layer="91"/>
+<label x="132.08" y="137.16" size="1.4224" layer="95" xref="yes"/>
+</segment>
+<segment>
+<pinref part="J6" gate="G$1" pin="2"/>
+<wire x1="200.66" y1="60.96" x2="213.36" y2="60.96" width="0.1524" layer="91"/>
+<label x="213.36" y="60.96" size="1.016" layer="95" xref="yes"/>
+</segment>
+</net>
+<net name="N$3" class="0">
+<segment>
+<pinref part="PCB1" gate="G$1" pin="GND@20"/>
+<wire x1="106.68" y1="116.84" x2="132.08" y2="116.84" width="0.1524" layer="91"/>
+<label x="132.08" y="116.84" size="1.778" layer="95" xref="yes"/>
+</segment>
+</net>
+<net name="D-" class="0">
 <segment>
 <pinref part="X1" gate="G$1" pin="2"/>
 <wire x1="121.92" y1="33.02" x2="134.62" y2="33.02" width="0.1524" layer="91"/>
 <label x="134.62" y="33.02" size="1.4224" layer="95" xref="yes"/>
-</segment>
-</net>
-<net name="GPS_CLK" class="0">
-<segment>
-<pinref part="U14" gate="G$1" pin="1PPS"/>
-<wire x1="210.82" y1="144.78" x2="226.06" y2="144.78" width="0.1524" layer="91"/>
-<label x="226.06" y="144.78" size="1.4224" layer="95" xref="yes"/>
-</segment>
-<segment>
-<pinref part="PCB1" gate="G$1" pin="GPIO24"/>
-<wire x1="106.68" y1="121.92" x2="132.08" y2="121.92" width="0.1524" layer="91"/>
-<label x="132.08" y="121.92" size="1.4224" layer="95" xref="yes"/>
-</segment>
-</net>
-<net name="ENABLE1" class="0">
-<segment>
-<pinref part="PCB1" gate="G$1" pin="GPIO18"/>
-<wire x1="106.68" y1="137.16" x2="132.08" y2="137.16" width="0.1524" layer="91"/>
-<label x="132.08" y="137.16" size="1.4224" layer="95" xref="yes"/>
-</segment>
-<segment>
-<pinref part="J6" gate="G$1" pin="2"/>
-<wire x1="200.66" y1="60.96" x2="213.36" y2="60.96" width="0.1524" layer="91"/>
-<label x="213.36" y="60.96" size="1.016" layer="95" xref="yes"/>
 </segment>
 </net>
@@
 <text x="114.3" y="137.16" size="2.54" layer="97">FTDI : USB (Pi) to Serial (GPS Receiver)</text>
 <text x="10.16" y="137.16" size="2.54" layer="97">Mother Board connector</text>
+<text x="119.38" y="93.98" size="2.54" layer="97">SDR (Socket Connector)</text>
 </plain>
 <instances>
@@
 <attribute name="NAME" x="32.004" y="109.728" size="1.778" layer="95" font="vector"/>
 <attribute name="VALUE" x="32.258" y="98.298" size="1.778" layer="96" font="vector" align="top-left"/>
+</instance>
+<instance part="J7" gate="G$1" x="134.62" y="106.68" smashed="yes">
+<attribute name="VALUE" x="129.54" y="99.314" size="1.778" layer="96" font="vector"/>
+<attribute name="NAME" x="129.54" y="114.808" size="1.778" layer="95" font="vector"/>
 </instance>
 </instances>
@@
 <label x="33.02" y="160.02" size="1.778" layer="95"/>
 </segment>
+<segment>
+<pinref part="J7" gate="G$1" pin="4"/>
+<wire x1="139.7" y1="111.76" x2="144.78" y2="111.76" width="0.1524" layer="91"/>
+<label x="144.78" y="111.76" size="1.778" layer="95"/>
+</segment>
 </net>
 <net name="TXO" class="0">
@@
 <label x="33.02" y="167.64" size="1.778" layer="95"/>
 </segment>
+<segment>
+<pinref part="J7" gate="G$1" pin="1"/>
+<wire x1="139.7" y1="104.14" x2="144.78" y2="104.14" width="0.1524" layer="91"/>
+<label x="144.78" y="104.14" size="1.778" layer="95"/>
+</segment>
 </net>
 <net name="D2-" class="0">
@@
 </segment>
 </net>
+<net name="D-" class="0">
+<segment>
+<pinref part="J7" gate="G$1" pin="2"/>
+<wire x1="139.7" y1="106.68" x2="144.78" y2="106.68" width="0.1524" layer="91"/>
+<label x="144.78" y="106.68" size="1.778" layer="95"/>
+</segment>
+</net>
+<net name="D+" class="0">
+<segment>
+<pinref part="J7" gate="G$1" pin="3"/>
+<wire x1="139.7" y1="109.22" x2="144.78" y2="109.22" width="0.1524" layer="91"/>
+<label x="144.78" y="109.22" size="1.778" layer="95"/>
+</segment>
+</net>
